Commit message: Added effort limits per joint to make it less bouncy

File: models/canadarm/urdf/SSRMS_Canadarm2.urdf.xacro (robot description, xacro)
@@ -10,4 +10,13 @@
   <xacro:include filename="$(find simulation)/models/canadarm/urdf/SSRMS_Canadarm2.gazebo.xacro" />
   <xacro:ssrms_canadarm2_gazebo command_interface="position" />
+  <!--Constant parameters-->
+  <!-- Default effort was 2332 for all joints -->
+  <xacro:property name="base_joint_effort"        value="8000.0" />
+  <xacro:property name="shoulder_roll_effort"        value="6000.0" />
+  <xacro:property name="shoulder_yaw_effort"        value="6000.0" />
+  <xacro:property name="elbow_pitch_effort"        value="4000.0" />
+  <xacro:property name="wrist_pitch_effort"        value="2332.0" />
+  <xacro:property name="wrist_yaw_effort"        value="2332.0" />
+  <xacro:property name="wrist_roll_effort"        value="2332.0" />
   <link name="world" />
   <joint name="world_joint" type="fixed">
@@ -44,5 +53,5 @@
     <origin rpy="0 0 0" xyz="0 0 0"/>
     <axis xyz="0 0 1"/>
-    <limit lower="-4.71239" upper="4.71239" effort="2332" velocity="0.0698132"/>
+    <limit lower="-4.71239" upper="4.71239" effort="${base_joint_effort}" velocity="0.0698132"/>
   </joint>
   <!--Manipulator-->
@@ -73,5 +82,5 @@
     <origin rpy="0 0 0" xyz="0.25082 0 -0.175"/>
     <axis xyz="1 0 0"/>
-    <limit lower="-4.71239" upper="4.71239" effort="2332" velocity="0.0698132"/>
+    <limit lower="-4.71239" upper="4.71239" effort="${shoulder_roll_effort}" velocity="0.0698132"/>
   </joint>
   <!-- Link 2 -->
@@ -101,5 +110,5 @@
     <origin rpy="0 0 0" xyz="0.175 0 -0.25082"/>
     <axis xyz="0 0 1"/>
-    <limit lower="-4.71239" upper="4.71239" effort="2332" velocity="0.0698132"/>
+    <limit lower="-4.71239" upper="4.71239" effort="${shoulder_yaw_effort}" velocity="0.0698132"/>
   </joint>
   <!-- Link 3 -->
@@ -159,5 +168,5 @@
     <origin rpy="0 0 0" xyz="7.61164 0 -0.6"/>
     <axis xyz="0 0 1"/>
-    <limit lower="-4.71239" upper="4.71239" effort="2332" velocity="0.0698132"/>
+    <limit lower="-4.71239" upper="4.71239" effort="${elbow_pitch_effort}" velocity="0.0698132"/>
   </joint>
   <!-- Link 5 -->
@@ -211,5 +220,5 @@
     <origin rpy="0 0 0" xyz="-7.61164 0 -0.35"/>
     <axis xyz="0 0 -1"/>
-    <limit lower="-4.71239" upper="4.71239" effort="2332" velocity="0.0698132"/>
+    <limit lower="-4.71239" upper="4.71239" effort="${wrist_pitch_effort}" velocity="0.0698132"/>
   </joint>
   <!-- Link 6 -->
@@ -239,5 +248,5 @@
     <origin rpy="0 0 0" xyz="-0.175 0 -0.25082"/>
     <axis xyz="1 0 0"/>
-    <limit lower="-4.71239" upper="4.71239" effort="2332" velocity="0.0698132"/>
+    <limit lower="-4.71239" upper="4.71239" effort="${wrist_yaw_effort}" velocity="0.0698132"/>
   </joint>
   <!-- Link 7 -->
@@ -267,5 +276,5 @@
     <origin rpy="0 0 0" xyz="-0.25082 0 -0.175"/>
     <axis xyz="0 0 1"/>
-    <limit lower="-4.71239" upper="4.71239" effort="2332" velocity="0.0698132"/>
+    <limit lower="-4.71239" upper="4.71239" effort="${wrist_roll_effort}" velocity="0.0698132"/>
   </joint>
   <!-- Link 8 -->
