Commit message: adding gateway like setup, adding camera to ee of ssrms

File: models/canadarm/urdf/SSRMS_Canadarm2.gazebo.xacro (robot description, xacro)
@@ -55,4 +55,28 @@
       <parameters>$(find canadarm)/config/canadarm_control.yaml</parameters>
       </plugin>
+      <plugin filename="ignition-gazebo-sensors-system" name="ignition::gazebo::systems::Sensors">
+      <background_color>0.0 0.0 0.0</background_color>
+      <render_engine>ogre2</render_engine>
+      </plugin>
+  </gazebo>
+  <gazebo reference="ee_camera">
+      <sensor type="camera" name="camera_sensor">
+          <pose>0 0 0 3.14 0 0</pose>
+          <visualize>1</visualize>
+          <update_rate>10.0</update_rate>
+          <camera>
+              <image>
+                  <width>800</width>
+                  <height>800</height>
+                  <format>R8G8B8</format>
+              </image>
+              <noise>
+              <type>gaussian</type>
+              <stddev>0.007</stddev>
+              </noise>
+          </camera>
+          <always_on>1</always_on>
+          <topic>image_raw</topic>
+      </sensor>
   </gazebo>
   <!-- Colors -->

File: models/canadarm/urdf/SSRMS_Canadarm2.urdf.xacro (robot description, xacro)
@@ -289,3 +289,13 @@
     </collision>
   </link>
+  <!-- Camera Joint: ee to camera -->
+  <joint name="ee_to_camera" type="fixed">
+    <parent link="EE_SSRMS"/>
+    <child link="ee_camera"/>
+    <origin rpy="0 1.570 0" xyz="-0.30 0.0 -1.15"/>
+    <axis xyz="0 0 1"/>
+    <limit lower="0" upper="0" effort="0" velocity="0"/>
+  </joint>
+  <!-- camera link -->
+  <link name="ee_camera"/>
 </robot>

Commit message: adding some cameras to candarm and a moon model

File: models/canadarm/urdf/SSRMS_Canadarm2.gazebo.xacro (robot description, xacro)
@@ -55,4 +55,29 @@
       <parameters>$(find canadarm)/config/canadarm_control.yaml</parameters>
       </plugin>
+      <plugin filename="ignition-gazebo-sensors-system" name="ignition::gazebo::systems::Sensors">
+        <background_color>0.0 0.0 0.0</background_color>
+        <render_engine>ogre2</render_engine>
+    </plugin>
+  </gazebo>
+  <gazebo reference="ee_camera">
+      <sensor type="camera" name="camera_sensor">
+          <pose>0 0 0 3.14 0 0</pose>
+          <visualize>1</visualize>
+          <update_rate>10.0</update_rate>
+          <camera>
+              <!-- <horizontal_fov>1.3962634</horizontal_fov> -->
+              <image>
+                  <width>800</width>
+                  <height>800</height>
+                  <format>R8G8B8</format>
+              </image>
+              <noise>
+              <type>gaussian</type>
+              <stddev>0.007</stddev>
+              </noise>
+          </camera>
+          <always_on>1</always_on>
+          <topic>image_raw</topic>
+      </sensor>
   </gazebo>
   <!-- Colors -->

File: models/canadarm/urdf/SSRMS_Canadarm2.urdf.xacro (robot description, xacro)
@@ -289,3 +289,13 @@
     </collision>
   </link>
+  <!-- Joint 7: Wrist Roll Joint -->
+  <joint name="ee_to_camera" type="fixed">
+    <parent link="EE_SSRMS"/>
+    <child link="ee_camera"/>
+    <origin rpy="0 1.570 0" xyz="-0.30 0.0 -1.15"/>
+    <axis xyz="0 0 1"/>
+    <limit lower="0" upper="0" effort="0" velocity="0"/>
+  </joint>
+  <!-- camera link -->
+  <link name="ee_camera"/>
 </robot>
